Commit message: Deleting gazebo color references

File: urdf/my_robot.xacro (robot description, xacro)
@@ -101,12 +101,6 @@
     </visual>
   </link>
-    <gazebo reference="left_wheel">
-    <material>Gazebo/Blue</material>
-  </gazebo>
-  <gazebo reference="right_wheel">
-    <material>Gazebo/Red</material>
-  </gazebo>
   <joint type="continuous" name="left_wheel_hinge">
-    <origin xyz="0 0.325 0" rpy="0 0 0" />
+    <origin xyz="0 0.15 0" rpy="0 0 0" />
     <child link="left_wheel" />
     <parent link="chassis" />
@@ -116,5 +110,5 @@
   </joint>
   <joint type="continuous" name="right_wheel_hinge">
-    <origin xyz="0 -0.325 0" rpy="0 0 0" />
+    <origin xyz="0 -0.15 0" rpy="0 0 0" />
     <child link="right_wheel" />
     <parent link="chassis" />

Commit message: Add camera sensor to my_robot.xacro

File: urdf/my_robot.xacro (robot description, xacro)
@@ -117,3 +117,33 @@
     <dynamics damping="1.0" friction="1.0" />
   </joint>
+  <link name="camera">
+    <inertial>
+      <mass value="0.1" />
+      <origin xyz="0 0 0" rpy="0 0 0" />
+      <inertia
+        ixx="1e-6" ixy="0" ixz="0"
+        iyy="1e-6" iyz="0"
+        izz="1e-6"
+      />
+    </inertial>
+    <box_inertia x="0.05" y="0.05" z="0.05" m="0.1" />
+    <collision>
+      <origin xyz="0 0 0" rpy="0 0 0" />
+      <geometry>
+        <box size="0.05 0.05 0.05"/>
+      </geometry>
+    </collision>
+    <visual>
+      <origin xyz="0 0 0" rpy="0 0 0" />
+      <geometry>
+        <box size="0.05 0.05 0.05"/>
+      </geometry>
+    </visual>
+  </link>
+  <joint type="fixed" name="camera_joint">
+    <origin xyz="0.2 0 0" rpy="0 0 0" />
+    <child link="camera" />
+    <parent link="chassis" />
+    <axis xyz="0 1 0" rpy="0 0 0" />
+  </joint>
 </robot>

Commit message: Changing colors and adding pluggin

File: urdf/my_robot.xacro (robot description, xacro)
@@ -1,4 +1,5 @@
 <?xml version='1.0'?>
 <robot name="my_robot" xmlns:xacro="http://www.ros.org/wiki/xacro">
+  <xacro:include filename="$(find my_robot)/urdf/my_robot.gazebo" />
   <link name="robot_footprint"></link>
   <joint name="robot_footprint_joint" type="fixed">
@@ -147,3 +148,47 @@
     <axis xyz="0 1 0" rpy="0 0 0" />
   </joint>
+  <link name="hokuyo">
+    <inertial>
+      <mass value="1e-5" />
+      <origin xyz="0 0 0" rpy="0 0 0" />
+      <inertia
+        ixx="1e-6" ixy="0" ixz="0"
+        iyy="1e-6" iyz="0"
+        izz="1e-6"
+      />
+    </inertial>
+    <collision>
+      <origin xyz="0 0 0" rpy="0 0 0" />
+      <geometry>
+        <box size="0.1 0.1 0.1"/>
+      </geometry>
+    </collision>
+    <visual>
+      <origin xyz="0 0 0" rpy="0 0 0" />
+      <geometry>
+        <mesh filename="package://my_robot/meshes/hokuyo.dae"/>
+      </geometry>
+    </visual>
+  </link>
+  <joint type="fixed" name="hokuyo_joint">
+    <origin xyz="0.15 0 0.1" rpy="0 0 0" />
+    <child link="hokuyo" />
+    <parent link="chassis" />
+    <axis xyz="0 1 0" rpy="0 0 0" />
+  </joint>
+  <gazebo reference = "chassis">
+    <material>Gazebo/Red</material>
+  </gazebo>
+  <gazebo reference = "right_wheel">
+    <material>Gazebo/Blue</material>
+  </gazebo>
+  <gazebo reference = "left_wheel">
+    <material>Gazebo/Blue</material>
+  </gazebo>
+  <gazebo reference = "hokuyo">
+    <material>Gazebo/Black</material>
+  </gazebo>
+  <gazebo reference = "camera">
+    <material>Gazebo/Green</material>
+  </gazebo>
 </robot>
